File: Circuit Schematics/Power and Regulation/Power and Regulation.kicad_sch (KiCad schematic)
At the start: 25 parts

Commit message: Whole boatload of changes
Latest.
Parts:
- removed C?: 10u, symbol Device:C_Small
- removed PFET? (x2): ECH8654, symbol ECH8654-TL-H_PFET:ECH8654
- removed Q?: FDS9926A, Package_SO:SOIC-8_3.9x4.9mm_P1.27mm, symbol Transistor_FET:FDS9926A
- removed U?: NTR3A052PZT1G, symbol NTR3A052PZT1G:NTR3A052PZT1G
- added C? (x2): 1u, symbol Device:C_Small
- added Q? (x2): DMG2302U, Package_TO_SOT_SMD:SOT-23, symbol Transistor_FET:DMG2302U
- added R?: 2.2k, symbol Device:R_Small_US
- added R?: 10k, symbol Device:R_US
- added R? (x2): 4.7k, symbol Device:R_US
- added U?: NCP163ASN330T1G, Package_TO_SOT_SMD:SOT-23-5, symbol Regulator_Linear:NCP163ASN330T1G
- added U? (x2): NTR3A052PZT1G, symbol NTR3A052PZT1G:NTR3A052PZT1G
- C1: value 1u -> 10u
Connections:
- net DIGI_ENABLE is gone; now on an unnamed net: VREG1.3 (~{SHDN})
- net +3V3: no longer C1.1, C2.2, VREG1.5 (OUT)
- net GND: now also C1.2, C1.2, C?.2, C?.2, SWIT?.1 (C), VREG1.2 (GND), VREG?.2 (GND), C?.2, C?.2, Q?.2 (S), R?.1, R?.2, U?.2 (GND)
- net GNDA: now also Q?.2 (S)
- net PICO_PWR: now also C1.1, C2.2, VREG1.5 (OUT), C?.1, R?.1, U?.2 (S), U?.5 (VOUT); no longer C1.1, VREG1.1 (IN)
- net ANA_BAT: now reaches C?.1, PFET?.5/6 (D), VREG?.1 (IN), VREG?.3 (~{SHDN})
- net at PFET?.4 (G), R1.1: now also Q?.3 (D)
- net at L1.1: now also Q?.1 (G)
- net at D?.1 (A), R1.1: now also U?.1 (G)
- net at V3xAA1.2-1.5V.1 (+): now also U?.3 (D)
- net at D?.3 (K): now also SWIT?.3 (C), U?.2 (S); no longer SWIT?.1 (C)
- net at SWIT?.2 (B): now also C1.1, VREG1.1 (IN), C?.1, R?.1, R?.1, U?.1 (VIN)
- new net: R?.2, U?.3 (EN)
- new net: Q?.3 (D), R?.2, U?.1 (G)
- new net 3V3_DIGITAL: U?.3 (D)
- new net DIGI_CON: Q?.1 (G), R?.2
Other:
- note added: "Digital Regulator"
- note added: "Digital Regulator (NCP163 onsemi rendition) (ver. 5. PCB) (250 mA limit)"
- note added: "Load Switch for Digi 3V3 (DIGI_CON HIGH TO POWER.)"
- note added: "NOTE! We've replaced ECH with NTR here. Now, remove the digital switch stuff! Just use a switch without a mosfet"
- note removed: "Digital Regulator w/ SHDN pin to Pico + PICO_PWR straight from battery"
- note removed: "General note for the technicalities/physicalities of configuring the Pico: - Connect MicroUSB to the device when it is turned OFF or recently turned ON (last minute or so.) - For the first minute-or-so, the device will ping to check if the USB VBUS sense pin is high. - If the USB VBUS sense pin is low/off, then the MicroUSB is not detected, + it waits for data logging w/ digital/analogue turned o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"
- note removed: "MicroUSB: - VBUS = VSYS - Gate = Source - MOSFET is closed + PICO_PWR disconnected - Body diode prevents current backflow"
- note removed: "No MicroUSB: - VBUS = 0, VSYS = 0 initially - Gate = Source - Body diode allows voltage through though - This raises VSYS - Gate - Source becomes negative - Opens MOSFET + VSYS = PICO_PWR"
- moved on the sheet: C1, C2, C?, D?, L1, PFET?, R1, R2, R?, SWIT?, V3xAA1.2-1.5V, V3xAA1.2-1.5V?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
