File: Circuit Schematics/Analogue Circuitry/Analogue Circuitry/Analogue Circuitry.kicad_sch (KiCad schematic)
At the start: 29 parts

Commit message: Whole boatload of changes
Latest.
Parts:
- removed C1: 0.1u, symbol Device:C_Small
- removed C2: 10u, symbol Device:C_Polarized_Small_US
- removed C3 (x2): 1u, symbol Device:C_Small
- removed C?: .1u, symbol Device:C_Small
- removed C_INA1, C_INA2: 4.7u, symbol Device:C_Small
- removed R? (x3): 10k, symbol Device:R_US
- removed R?: 10k, symbol Device:R_Small_US
- removed R_BOT: 68k, symbol Device:R_Small_US
- removed R_TOP: 55.6k, symbol Device:R_Small_US
- removed VR2: MCP4131-103E/SN, SOIC127P599X175-8N, symbol MCP4131-103E_SN:MCP4131-103E/SN
- removed VREF2: MAX6070, symbol MAX6070:MAX6070
- added C? (x2): 10u, symbol Device:C_Polarized_Small_US
- added C? (x2): 1u, symbol Device:C_Small
- added C?: 0.1u, symbol Device:C_Small
- added C? (x2): 10u, symbol Device:C_Small
- added R? (x7): 10k, symbol Device:R_US
- added R?: 100, symbol Device:R_Small_US
- added R? (x3): 1k, symbol Device:R_US
- added R? (x2): 22k, symbol Device:R_US
- added R?: 330, symbol Device:R_Small_US
- C3: value 1u -> 10u
Connections:
- net REF_OUTS is gone; now on net 3V3_VREF: VREF1.5 (OUTS)
- net +3V3: no longer C3.1, R?.2, VREF1.4 (IN)
- net CASCADE_OUT: now also VR1.6 (P0W); no longer VR1.7 (P0B)
- net GNDA: now also C?.1, C?.2, C?.2, C?.2, C?.2, R?.2, R?.2
- net SCK_VR: now also R?.2
- net SDIO_VR: now also R?.2
- net at OPAMP1-2.5 (INB+): now also C?.1, R?.1, R?.2; no longer OPAMP1-2.3 (INA+)
- net at C1.1, OPAMP1-2.1 (OUTA): now also R?.2
- net at C1.2: now also R?.1; no longer VR1.5 (P0A)
- net at OPAMP1-2.6 (INB-): now also VR1.5 (P0A), R?.2; no longer VR1.6 (P0W)
- net at MIC1.1 (OUT+): now also C?.1
- net at OPAMP1-2.2 (INA-): now also R?.1, R?.2
- net at MIC1.6 (OUT-): now also C?.1
- net Analogue Regulator: no longer names the net of MIC1.5 (VDD)
- net Analogue Regulator: now also R?.2; no longer OPAMP1-2.8 (VDD)
- net CS_VR1 renamed CS_VR
- net CS_VR: now also R?.2
- net GNDD renamed 3V3_DIGI
- net 3V3_DIGI: now also R?.1, R?.1, R?.1
- net REF_OUTF renamed 3V3_VREF
- net 3V3_VREF: now also C?.1, C?.1, R?.1, R?.1
- new net: C?.2, R?.1 (x2)
- new net: C?.1, R?.1, R?.1, R?.2
- new net: C3.1, R?.2, R?.2, VREF1.4 (IN)
- new net: OPAMP1-2.3 (INA+), R?.2, R?.2
- new net 3V3_ANA: C?.2, OPAMP1-2.8 (VDD), R?.1
- new net ANA_BAT: R?.1
Other:
- note added: "Bias of 3V/2"
- note added: "Multiplexed SDIO Stuff ====================== See https://electronics.stackexchange.com/ questions/240852/mcp4131-how-to-know-what- value-resistors-to-use-on-the-multiplexed- spi-io to decide on value of R here. Let the worst low-level be about 0.5V like they say Input leakage is 1 muA Input MCU leakage is around 1-2 muA Maximum voltage for low is about 0.7V Use an R1 = 4.7k and get an R2 of abou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"
- note added: "See the LTSpice file Draft2 for the best example."
- note added: "Use the digipot as a varistor for R2 on the inverting 2nd stage."
- note removed: "Bias to 3V3/2. Use voltage dividers. Pico with 3V on the VREF will need 3V/2 biasing."
- note removed: "Design note C1/C2 ================= AC coupling capacitor (removes DC) Specifies a high-pass Use formula (find) Get corner freq. 7-8 kHz recommended highpass."
- note removed: "Design note additions: - see https://www.reddit.com/r/ElectricalEngineering/comments/1002wz0/pcb_design_considerations_for_a_cascaded/ - we're replacing our arrangement - fix the gain of the first op-amp stage: we need to decide on which fix, but yeah. - set the gain on the second stage to be variable. - we can make the first stage a differential amplifier, which will minimize noise on traces fro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"
- note removed: "Divider 3V MAX6070. Use 50k:50k for 3V3 MAX6070."
- note removed: "GAIN_1=-R2/R1"
- note removed: "GAIN_2=-R4/R3"
- note removed: "INCLUDE PULLUPS ON THE SDIO AND SCK LINES! FUCKER! AND THE FUCKING CSN!"
- note removed: "Potentiometer -> R1 & R2"
- note removed: "Potentiometer -> R3 & R4"
- note removed: "Quick design note ================= Microchip do a dual-pot model. Others do too. Replace with dual-pot model for final production. Might need to consider cross-talk if you use a dual. Check possibilities. As of the moment, dual pot Microchip is unavailable."
- note removed: "Quick design note ================= This model is 3-line SPI. Might be troublesome to implement. Shared MOSI/MISO. Diodes!!!"
- note removed: "REPLACE MAX6070 3V WITH 3V3 ONCE WE HAVE USED UP 3V!"
- note removed: "See https://electronics.stackexchange.com/questions/240852/mcp4131-how-to-know-what-value-resistors-to-use-on-the-multiplexed-spi-io to decide on value of R here. Let the worst low-level be about 0.5V like they say Input leakage is 1 muA Input MCU leakage is around 1-2 muA Maximum voltage for low is about 0.7V Use an R1 = 4.7k and get an R2 of about 68k (or close-enough) for pullup"
- note removed: "Solder note: skip soldering OUT-. Makes reflow difficult."
- note removed: "To ADC"
- note removed: "Variable Gain SPI Potentiometers"
- moved on the sheet: C1, C3, MIC1, OPAMP1-2, R1, R2, R?, V2, VR1, VREF1

Commit message: 1
1
Parts:
- added C? (x2): C, symbol Device:C
Connections:
- net 3V3_DIGI: now also C?.1
- net at MIC1.5 (VDD), R?.2: now also C?.2
- new net GNDD: C?.1, C?.2
Changed lines of the file:
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@@
   (junction (at 109.22 153.67) (diameter 0) (color 0 0 0 0)
   )
+  (junction (at 140.97 46.99) (diameter 0) (color 0 0 0 0)
+  )
   (junction (at 71.12 120.65) (diameter 0) (color 0 0 0 0)
   )
@@
   )
   (junction (at 137.16 59.69) (diameter 0) (color 0 0 0 0)
+  )
+  (junction (at 30.48 135.89) (diameter 0) (color 0 0 0 0)
   )
   (junction (at 137.16 46.99) (diameter 0) (color 0 0 0 0)
@@
     (stroke (width 0) (type default) (color 0 0 0 0))
   )
+  (wire (pts (xy 140.97 46.99) (xy 143.51 46.99))
+    (stroke (width 0) (type default) (color 0 0 0 0))
+  )
   (wire (pts (xy 107.95 153.67) (xy 109.22 153.67))
     (stroke (width 0) (type default) (color 0 0 0 0))
@@
     (stroke (width 0) (type default) (color 0 0 0 0))
   )
-  (wire (pts (xy 137.16 46.99) (xy 143.51 46.99))
+  (wire (pts (xy 137.16 46.99) (xy 140.97 46.99))
     (stroke (width 0) (type default) (color 0 0 0 0))
   )
@@
     (pin "2")
   )
+  (symbol (lib_id "power:GNDD") (at 140.97 54.61 0) (unit 1)
+    (in_bom yes) (on_board yes) (fields_autoplaced)
+    (property "Reference" "#PWR?" (id 0) (at 140.97 60.96 0)
+      (effects (font (size 1.27 1.27)) hide)
+    )
+    (property "Value" "GNDD" (id 1) (at 140.97 59.69 0))
+    (property "Footprint" "" (id 2) (at 140.97 54.61 0)
+      (effects (font (size 1.27 1.27)) hide)
+    )
+    (property "Datasheet" "" (id 3) (at 140.97 54.61 0)
+      (effects (font (size 1.27 1.27)) hide)
+    )
+    (pin "1")
+  )
+  (symbol (lib_id "power:GNDD") (at 30.48 128.27 180) (unit 1)
+    (in_bom yes) (on_board yes) (fields_autoplaced)
+    (property "Reference" "#PWR?" (id 0) (at 30.48 121.92 0)
+      (effects (font (size 1.27 1.27)) hide)
+    )
+    (property "Value" "GNDD" (id 1) (at 33.02 127.1904 0)
+      (effects (font (size 1.27 1.27)) (justify right))
+    )
+    (property "Footprint" "" (id 2) (at 30.48 128.27 0)
+      (effects (font (size 1.27 1.27)) hide)
+    )
+    (property "Datasheet" "" (id 3) (at 30.48 128.27 0)
+      (effects (font (size 1.27 1.27)) hide)
+    )
+    (pin "1")
+  )
   (symbol (lib_id "Device:C_Polarized_Small_US") (at 54.61 134.62 180) (unit 1)
     (in_bom yes) (on_board yes)
@@
     (pin "2")
   )
+  (symbol (lib_id "Device:C") (at 140.97 50.8 0) (unit 1)
+    (in_bom yes) (on_board yes) (fields_autoplaced)
+    (property "Reference" "C?" (id 0) (at 144.78 49.5299 0)
+      (effects (font (size 1.27 1.27)) (justify left))
+    )
+    (property "Value" "C" (id 1) (at 144.78 52.0699 0)
+      (effects (font (size 1.27 1.27)) (justify left))
+    )
+    (property "Footprint" "" (id 2) (at 141.9352 54.61 0)
+      (effects (font (size 1.27 1.27)) hide)
+    )
+    (property "Datasheet" "~" (id 3) (at 140.97 50.8 0)
+      (effects (font (size 1.27 1.27)) hide)
+    )
+    (pin "1")
+    (pin "2")
+  )
   (symbol (lib_id "Device:C_Small") (at 205.74 64.77 0) (unit 1)
     (in_bom yes) (on_board yes) (fields_autoplaced)
@@
     (pin "2")
   )
+  (symbol (lib_id "Device:C") (at 30.48 132.08 0) (unit 1)
+    (in_bom yes) (on_board yes) (fields_autoplaced)
+    (property "Reference" "C?" (id 0) (at 34.29 130.8099 0)
+      (effects (font (size 1.27 1.27)) (justify left))
+    )
+    (property "Value" "C" (id 1) (at 34.29 133.3499 0)
+      (effects (font (size 1.27 1.27)) (justify left))
+    )
+    (property "Footprint" "" (id 2) (at 31.4452 135.89 0)
+      (effects (font (size 1.27 1.27)) hide)
+    )
+    (property "Datasheet" "~" (id 3) (at 30.48 132.08 0)
+      (effects (font (size 1.27 1.27)) hide)
+    )
+    (pin "1")
+    (pin "2")
+  )
   (sheet_instances
     (path "/" (page "1"))
@@
       (reference "#PWR?") (unit 1) (value "GNDA") (footprint "")
     )
+    (path "/3dc4af7e-fb9d-4b46-8986-9ab4081fc304"
+      (reference "#PWR?") (unit 1) (value "GNDD") (footprint "")
+    )
+    (path "/3e32c059-9625-4611-9346-af15caae75d1"
+      (reference "#PWR?") (unit 1) (value "GNDD") (footprint "")
+    )
     (path "/4875f367-a3ed-476b-8963-592f8549b23a"
       (reference "#PWR?") (unit 1) (value "GNDA") (footprint "")
@@
       (reference "C?") (unit 1) (value "10u") (footprint "")
     )
+    (path "/bb02af3e-6599-4e65-886b-fc630b83c217"
+      (reference "C?") (unit 1) (value "C") (footprint "")
+    )
     (path "/c4255389-7e49-4a5b-810e-1973c67e5bda"
       (reference "C?") (unit 1) (value "1u") (footprint "")
@@
       (reference "C?") (unit 1) (value "10u") (footprint "")
     )
+    (path "/ff666e32-b1b1-4049-95b6-190e17bcb1e5"
+      (reference "C?") (unit 1) (value "C") (footprint "")
+    )
     (path "/c9724bf5-d828-4fcf-b304-bc41143bc620"

Commit message: Bunch of changes
and I'm a lazy mofo who doesn't want to version control my directory and so yeah
Parts:
- added C2: 390pF, symbol Device:C_Small
- added C3: 180, symbol Device:C_Small
- added C4: 100p, symbol Device:C_Small
- added C?: 0.1u, symbol Device:C_Small
- added C? (x2): 10u, symbol Device:C_Small
- added C? (x3): 10u, symbol Device:C_Polarized_Small_US
- added C?: C, symbol Device:C
- added C? (x2): 1u, symbol Device:C_Small
- added MIC?: SPM0687LR5H-1, symbol SPM0687LR5H-1:SPM0687LR5H-1
- added O?: OPA, Package_SON:Texas_S-PVSON-N10, symbol Amplifier_Audio:OPA1622
- added OPAMP1-?: MAX40089AUA+, 21-0036K_MXM, symbol MAX40089AUA+:MAX40089AUA+
- added PGA_1: PGA, symbol ADG812YRUZ:ADG812YRUZ
- added R? (x3): 1k, symbol Device:R_US
- added R? (x4), RP4: 10k, symbol Device:R_US
- added R? (x4): R_US, symbol Device:R_US
- added R? (x2): 22k, symbol Device:R_US
- added R?: 100, symbol Device:R_Small_US
- added RP1: 5k, symbol Device:R_US
- added RP2: 40k, symbol Device:R_US
- added RP3: 20k, symbol Device:R_US
- added V?: RIN, symbol Device:R_Small_US
- added V?: RF, symbol Device:R_Small_US
Connections:
- net +3V3: now also PGA_1.13 (VDD)
- net 3V3_ANA: now also C?.2, OPAMP1-?.8 (VDD), R?.1
- net 3V3_VREF: now also C?.1, C?.1, R?.1, R?.1
- net CASCADE_OUT: now also C2.1, C3.1, C4.1, OPAMP1-?.7 (OUTB), RP1.1, RP2.1, RP3.1, RP4.1
- net GNDA: now also C?.1, C?.2, C?.2, C?.2, C?.2, MIC?.2 (GND), MIC?.3 (GND), MIC?.4 (GND), O?.1 (+), OPAMP1-?.4 (VSS), R?.2, R?.2
- net GNDD: now also C?.1, PGA_1.5 (GND), R?.2, R?.2, R?.2, R?.2
- new net: O?.10 (-), V?.1, V?.2
- new net: O?.9, V?.2
- new net: C3.2, PGA_1.11 (S3), RP3.2
- new net: C?.1, OPAMP1-?.5 (INB+), R?.1, R?.2
- new net: C?.1, OPAMP1-?.1 (OUTA), R?.2
- new net: C?.2, R?.1 (x3)
- new net: C2.2, PGA_1.14 (S2), RP2.2
- new net: OPAMP1-?.3 (INA+), R?.2, R?.2
- new net: PGA_1.3 (S1), RP1.2
- new net: C?.2, MIC?.5 (VDD), R?.2
- new net: C?.1, MIC?.1 (OUT+)
- new net: C?.1, MIC?.6 (OUT-)
- new net: OPAMP1-?.2 (INA-), R?.1, R?.2
- new net: C4.2, PGA_1.6 (S4), RP4.2
- new net: OPAMP1-?.6 (INB-), PGA_1.10 (D3), PGA_1.15 (D2), PGA_1.2 (D1), PGA_1.7 (D4), R?.2
- new net: C?.1, R?.1, R?.1, R?.2
- new net PGA_1: PGA_1.8 (IN4), R?.1
- new net PGA_2: PGA_1.1 (IN1), R?.1
- new net PGA_3: PGA_1.16 (IN2), R?.1
- new net PGA_4: PGA_1.9 (IN3), R?.1
- no-connect marks 1 -> 3
Other:
- note added: "10k pulldown array"
- note added: "ANALOGUE SWITCH PGA EDITION 2ND STAGE GAIN OF: 5,10,20,40"
- note added: "D and S are interchangeable D1 and S1 are open when IN1 high Compensate appropriately!!!!"
- note added: "Drive whichever you want to logic high This closes appropriate switch"
- note added: "Four gains optional- 5,10,20,40. Note undercompensation. Note that you could combine two resistances in parallel- that results in overcompensation, however, attenuating higher frequencies a lot. I.e. if you open 5k and 10k at once, that's 10/3 gain- you then have overcompensation of 100 pF though. Using two PGAs one with caps one with R is an option- let's just try four gains first, though."
- note added: "Varistor here (variable gain.)"
